File: droidstamp_pcb_vsie2/STM32.sch (KiCad schematic (older format))
At the start: 51 parts, among them P6 CONN_5X2, P8 CONN_12X2, P9 CONN_12X2, Q2 BS170F, Q3 BS170F, Q4 BS170F, Q5 BS170F, Q6 BS170F, Q7 BS170F, Q8 BS170F, Q9 BS170F, U11 LT1117CST-3.3, U12 ZXMHC3F381N8, U13 ZXMHC3F381N8, U14 ZXMHC3F381N8, U15 ZXMHC3F381N8, U9 STM32F4_LQFP100, X3 12MHz

Commit message: EMF Feedback For M1 -- Incomplete. Must include module for SN74CBT1G125.
For the moment it is a 74LS125 which conceptually is somehow similar.
Parts:
- added C?: 1nF, symbol C
- added R? (x2): 10k, symbol R
- added R? (x2): 20k, symbol R
- added U? (x2): 74LS125, symbol 74LS125
Connections:
- net labels added: EMF_M1, EMF_M11, EMF_M12, PWM_C1M1, PWM_C2M1, SMPL_M11, SMPL_M12
- wire segments 257 -> 268
Other:
- note added: "74LS125 must be changed by SN74CBT1G125 or similar analog switch."
- moved on the sheet: R35, R37, U12

Commit message: Library for sn74cbt1g125. TODO: current sensing.
Parts:
- removed C?: 1nF, symbol C
- removed Q2: BS170F, BS170F, symbol MOSFET_N_OPENDOUS
- removed R35, R37: 2.2k, SM0603, symbol R
- removed U? (x2): 74LS125, symbol 74LS125
- added C?: 1nF, symbol C
- added L?: 1mH, symbol INDUCTOR
- added Q?: BS170F, BS170F, symbol MOSFET_N_OPENDOUS
- added R? (x4): 10, symbol R
- added R? (x2): 2.2k, symbol R
- added R? (x2): 100k, symbol R
- added U? (x2): SN74CBT1G125, -SOT23-5L, symbol SN74CBT1G125
Connections:
- net labels added: GMDMTR
- wire segments 268 -> 285
Other:
- note removed: "74LS125 must be changed by SN74CBT1G125 or similar analog switch."
- moved on the sheet: R?, U12

Commit message: Current sense for M1 -- taken from openservo.
Parts:
- added C?: 0.1uF, symbol C
- added R?: 0.05, symbol R
- added R?: 1k, symbol R
- added R?: 5k1, symbol R
- added U?: ZXCT1009, symbol ZXCT1009
Connections:
- net labels added: I_sense_M1, M1_torque_sense
- wire segments 285 -> 292

Commit message: Feedback for motors 1 and 2 in different sheet. Current feedback for M1 and M2.
Connection between digital ground and motor ground by means of an inductor.
Parts:
- removed C?: 1nF, symbol C
- removed Q3, Q4, Q5, Q?: BS170F, BS170F, symbol MOSFET_N_OPENDOUS
- removed R38, R39: 2.2k, SM0603, symbol R
- removed R? (x2): 10k, symbol R
- removed R? (x2): 20k, symbol R
- removed R? (x4): 10, symbol R
- removed R? (x2): 2.2k, symbol R
- removed R? (x2): 100k, symbol R
- removed U12, U13: ZXMHC3F381N8, -SO8, symbol ZXMHC3F381N8
- removed U? (x2): SN74CBT1G125, -SOT23-5L, symbol SN74CBT1G125
Connections:
- net labels removed: EMF_M1, EMF_M11, EMF_M12, PWM_C1M1, PWM_C2M1, SMPL_M11, SMPL_M12
- wire segments 292 -> 230
Other:
- moved on the sheet: C?, L?, P6, R40, R41, R44, R45, R?, U14, U15

Commit message: Current sensing separated in the feedback_drivers sheet.
Parts:
- removed C?: 0.1uF, symbol C
- removed L?: 1mH, symbol INDUCTOR
- removed R?: 0.05, symbol R
- removed R?: 1k, symbol R
- removed R?: 5k1, symbol R
- removed U?: ZXCT1009, symbol ZXCT1009
- added L?: 1mH, symbol INDUCTOR
Connections:
- net labels removed: I_sense_M1, M1_torque_sense
- wire segments 230 -> 223
Changed lines of the file:
@@
-EESchema Schematic File Version 2  date Thu 19 Apr 2012 07:33:46 PM EDT
+EESchema Schematic File Version 2  date Thu 19 Apr 2012 10:29:31 PM EDT
 LIBS:../components/con-jack,../components/zxct1009,../components/adm3101e,../components/microsd,../components/transistor-npn,../components/ipc-7351-transistor,../components/switch-misc,power,device,transistors,conn,linear,regul,74xx,cmos4000,adc-dac,memory,xilinx,special,microcontrollers,dsp,microchip,analog_switches,motorola,texas,intel,audio,interface,digital-audio,philips,display,cypress,siliconi,opto,atmel,contrib,valves,../components/micron_ddr_512Mb,../components/iMX23,../components/sdmmc,../components/usbconn,../components/fsusb20,../components/r_pack2,../components/pasives-connectors,../components/EEPROM,../components/PWR,../components/m25p32,../components/PROpendous-cache,../components/w_analog,../components/gl850g,../components/srf2012,../components/rclamp0502b,../components/mcp130,../components/ABM8G,../components/usb_a,../components/Reset,../components/stm32f100vxx,../components/lt1117cst,../components/zxmhc3f381n8,../components/stm32f4_lqfp100,./i.mx233stamp.cache
 EELAYER 24  0
@@
 Comment4 ""
 $EndDescr
+Wire Wire Line
+	7150 3250 7150 3200
+Wire Wire Line
+	7150 3200 7250 3200
+Wire Wire Line
+	7850 3200 8000 3200
+Text Label 8000 3200 0    60   ~ 0
+GMDMTR
+$Comp
+L GND #PWR?
+U 1 1 4F90C955
+P 7150 3250
+F 0 "#PWR?" H 7150 3250 30  0001 C CNN
+F 1 "GND" H 7150 3180 30  0001 C CNN
+	1    7150 3250
+	1    0    0    -1
+$EndComp
+$Comp
+L INDUCTOR L?
+U 1 1 4F90C954
+P 7550 3200
+F 0 "L?" V 7500 3200 40  0000 C CNN
+F 1 "1mH" V 7650 3200 40  0000 C CNN
+	1    7550 3200
+	0    -1   -1   0
+$EndComp
 $Sheet
 S 6900 3700 4550 1500
@@
 F1 "motors_feedback_drivers.sch" 60
 $EndSheet
-Text Label 2950 1150 0    60   ~ 0
-M1_torque_sense
-Wire Wire Line
-	2950 1150 2950 1300
-Wire Wire Line
-	2950 1700 3550 1700
-Wire Wire Line
-	3650 1250 3450 1250
-Wire Wire Line
-	5200 1700 5200 1450
-Wire Wire Line
-	5200 1450 4950 1450
-Wire Wire Line
-	3800 800  3800 750
-Wire Wire Line
-	3800 750  3900 750
 Wire Wire Line
 	-2500 7050 -2500 7000
@@
 Wire Wire Line
 	-400 1700 0    1700
-Wire Wire Line
-	4500 750  4650 750
-Wire Wire Line
-	5400 1050 4950 1050
-Wire Wire Line
-	3550 1700 3550 1800
-$Comp
-L GND #PWR?
-U 1 1 4F8E14C8
-P 3550 1800
-F 0 "#PWR?" H 3550 1800 30  0001 C CNN
-F 1 "GND" H 3550 1730 30  0001 C CNN
-	1    3550 1800
-	1    0    0    -1
-$EndComp
-$Comp
-L C C?
-U 1 1 4F8E14B7
-P 2950 1500
-F 0 "C?" H 3000 1600 50  0000 L CNN
-F 1 "0.1uF" H 3000 1400 50  0000 L CNN
-	1    2950 1500
-	1    0    0    -1
-$EndComp
-$Comp
-L R R?
-U 1 1 4F8E13BA
-P 3550 1500
-F 0 "R?" V 3630 1500 50  0000 C CNN
-F 1 "5k1" V 3550 1500 50  0000 C CNN
-	1    3550 1500
-	1    0    0    -1
-$EndComp
-$Comp
-L R R?
-U 1 1 4F8E13B5
-P 3200 1250
-F 0 "R?" V 3280 1250 50  0000 C CNN
-F 1 "1k" V 3200 1250 50  0000 C CNN
-	1    3200 1250
-	0    1    1    0
-$EndComp
-Text Label 5200 1700 0    60   ~ 0
-I_sense_M1
-Text Label 5400 1050 0    60   ~ 0
-VMTR
-$Comp
-L R R?
-U 1 1 4F8E135A
-P 5200 1300
-F 0 "R?" V 5280 1300 50  0000 C CNN
-F 1 "0.05" V 5200 1300 50  0000 C CNN
-	1    5200 1300
-	1    0    0    -1
-$EndComp
-$Comp
-L ZXCT1009 U?
-U 1 1 4F8E133F
-P 4300 1250
-F 0 "U?" H 4450 1250 60  0000 C CNN
-F 1 "ZXCT1009" H 4300 950 60  0000 C CNN
-	1    4300 1250
-	1    0    0    -1
-$EndComp
-Text Label 4650 750  0    60   ~ 0
-GMDMTR
-$Comp
-L GND #PWR?
-U 1 1 4F8D4182
-P 3800 800
-F 0 "#PWR?" H 3800 800 30  0001 C CNN
-F 1 "GND" H 3800 730 30  0001 C CNN
-	1    3800 800
-	1    0    0    -1
-$EndComp
-$Comp
-L INDUCTOR L?
-U 1 1 4F8D4176
-P 4200 750
-F 0 "L?" V 4150 750 40  0000 C CNN
-F 1 "1mH" V 4300 750 40  0000 C CNN
-	1    4200 750
-	0    -1   -1   0
-$EndComp
 $Comp
 L VDD5V #PWR?
