File: droidstamp_pcb_vsie2/motors_feedback_drivers.sch (KiCad schematic (older format))
At the start: 36 parts

Commit message: Current sensing separated in the feedback_drivers sheet.
Parts:
- added C? (x2): 0.1uF, symbol C
- added R? (x2): 0.05, symbol R
- added R? (x2): 1k, symbol R
- added R? (x2): 5k1, symbol R
- added U? (x2): ZXCT1009, symbol ZXCT1009
Connections:
- net labels added: M1_torque_sense, M2_torque_sense
- wire segments 88 -> 102
Other:
- moved on the sheet: C?, R?, U?
