File: droidstamp_pcb_lt/i.mx233stamp.sch (KiCad schematic (older format))
At the start: 0 parts

Commit message: ratnets revision
Connections:
- wire segments 32 -> 16
Changed lines of the file:
@@
-EESchema Schematic File Version 2  date Mon 18 Jun 2012 02:03:20 AM COT
+EESchema Schematic File Version 2  date Mon 18 Jun 2012 06:53:05 AM COT
 LIBS:con-jack
 LIBS:zxct1009
@@
 	3000 3650 3150 3650
 Wire Wire Line
-	2900 1850 3150 1850
-Wire Wire Line
-	2900 2700 3150 2700
-Wire Wire Line
-	3000 4150 3150 4150
-Wire Wire Line
-	2900 2450 3150 2450
-Wire Wire Line
-	2900 2350 3150 2350
-Wire Wire Line
-	2900 2150 3150 2150
-Wire Wire Line
-	3000 3950 3150 3950
-Wire Wire Line
-	3000 3750 3150 3750
-Wire Wire Line
 	3150 3450 3000 3450
 Wire Bus Line
@@
 Wire Wire Line
 	3000 3550 3150 3550
-Wire Wire Line
-	3000 3850 3150 3850
-Wire Wire Line
-	3000 4050 3150 4050
-Wire Wire Line
-	2900 2050 3150 2050
-Wire Wire Line
-	2900 2250 3150 2250
-Wire Wire Line
-	2900 2550 3150 2550
-Wire Wire Line
-	3000 4250 3150 4250
-Wire Wire Line
-	3150 2800 2900 2800
-Wire Wire Line
-	2900 1950 3150 1950
-$Sheet
-S 3150 1600 1600 2950
-U 4D30AC69
-F0 "i.MX233" 60
-F1 "i.MX233.sch" 60
-F2 "DDR_A[0..12]" O R 4750 2400 60
-F3 "DDR_DQ[0..15]" B R 4750 2500 60
-F4 "DDR_WEN" O R 4750 2750 60
-F5 "DDR_RASN" O R 4750 2950 60
-F6 "DDR_DQS1" O R 4750 3200 60
-F7 "DDR_DQS0" O R 4750 3100 60
-F8 "DDR_DQM1" O R 4750 3450 60
-F9 "DDR_DQM0" O R 4750 3350 60
-F10 "DDR_CLK" O R 4750 3600 60
-F11 "DDR_CLKN" O R 4750 3700 60
-F12 "DDR_CKE" O R 4750 3800 60
-F13 "DDR_CASN" O R 4750 2850 60
-F14 "DDR_CE0" O R 4750 2650 60
-F15 "DDR_BA1" O R 4750 4050 60
-F16 "DDR_BA0" O R 4750 3950 60
-F17 "USB_DM" B L 3150 3550 60
-F18 "USB_DP" B L 3150 3450 60
-F19 "USB_M3" B L 3150 4050 60
-F20 "USM_P3" B L 3150 3950 60
-F21 "USB_M4" B L 3150 3850 60
-F22 "USB_P4" B L 3150 3750 60
-F23 "I2C_SCL" B L 3150 2700 60
-F24 "I2C_SDA" B L 3150 2800 60
-F25 "GPMI_CE0N" B L 3150 2050 60
-F26 "SSPI_DETECT" B L 3150 2350 60
-F27 "GPMI_CE1N" B L 3150 2150 60
-F28 "GPMI_D06" B L 3150 2550 60
-F29 "SSPI_DATA3" B L 3150 2450 60
-F30 "USM_P2" B L 3150 4150 60
-F31 "USB_M2" B L 3150 4250 60
-F32 "AUART_TX" B L 3150 1950 60
-F33 "AUART_RX" B L 3150 1850 60
-F34 "PWM2" B L 3150 2250 60
-F35 "GPMI_D04" O L 3150 3650 60
-$EndSheet
 $Sheet
 S 5250 1600 1150 2500
@@
 F2 "USB_DM0" T R 3000 3550 60
 F3 "USB_DP0" T R 3000 3450 60
-F4 "USB_P4" B R 3000 3750 60
-F5 "USB_M4" B R 3000 3850 60
-F6 "USM_P3" B R 3000 3950 60
-F7 "USB_M3" B R 3000 4050 60
-F8 "USB_M2" B R 3000 4250 60
-F9 "USM_P2" B R 3000 4150 60
-F10 "USB_reset" B R 3000 3650 60
+F4 "USB_reset" B R 3000 3650 60
+$EndSheet
+$Sheet
+S 3150 1600 1600 2950
+U 4D30AC69
+F0 "i.MX233" 60
+F1 "i.MX233.sch" 60
+F2 "DDR_A[0..12]" O R 4750 2400 60
+F3 "DDR_DQ[0..15]" B R 4750 2500 60
+F4 "DDR_WEN" O R 4750 2750 60
+F5 "DDR_RASN" O R 4750 2950 60
+F6 "DDR_DQS1" O R 4750 3200 60
+F7 "DDR_DQS0" O R 4750 3100 60
+F8 "DDR_DQM1" O R 4750 3450 60
+F9 "DDR_DQM0" O R 4750 3350 60
+F10 "DDR_CLK" O R 4750 3600 60
+F11 "DDR_CLKN" O R 4750 3700 60
+F12 "DDR_CKE" O R 4750 3800 60
+F13 "DDR_CASN" O R 4750 2850 60
+F14 "DDR_CE0" O R 4750 2650 60
+F15 "DDR_BA1" O R 4750 4050 60
+F16 "DDR_BA0" O R 4750 3950 60
+F17 "USB_DM" B L 3150 3550 60
+F18 "USB_DP" B L 3150 3450 60
+F19 "GPMI_D04" O L 3150 3650 60
 $EndSheet
 $EndSCHEMATC
